File: hardware/Isolated Multi-Rail Power Supply Monitor Arduino Shield Board/Isolated Multi-Rail Power Supply Monitor Arduino Shield Board.kicad_sch (KiCad schematic)
At the start: 78 parts, among them J201 SI-46014-F, J309 0039289088, U202 W6100-Q, U4 TPS62912, U7 P82715DR, Y201 25MHz

Commit message: Nightly commit
Parts:
- added N101: Giga_Display, symbol Mechanical:Housing
- A201: value Arduino_Giga_R1_WiFi_Shield -> Arduino_Giga_R1_WiFi; DPN (none) -> 1050-ABX00063-ND; Distributor (none) -> Digikey; MPN (none) -> ABX00063; Manufacturer (none) -> Arduino; now in the parts list
- FB201, FB202, FB203: DPN 490-3996-6-ND -> 553-BBUP00160805121Y00CT-ND; MPN BLM18SG121TN1D -> BBUP00160805121Y00; Manufacturer Murata Electronics -> Pulse Electronics
- R205, R206, R207, R23, R24: DPN P4.70KLDKR-ND -> 541-4.70KLCT-ND; MPN ERJ-2RKF4701X -> CRCW04024K70FKED; Manufacturer Panasonic Industry -> Vishay Dale
- R21, R25, R26: DPN P4.70KLDKR-ND -> (none); MPN ERJ-2RKF4701X -> (none)
- TP1, TP101, TP3: DPN (none) -> 36-5000-ND; Distributor (none) -> Digikey; MPN (none) -> 5000; Manufacturer (none) -> Keystone
- TP102, TP2: DPN (none) -> 36-5001-ND; Distributor (none) -> Digikey; MPN (none) -> 5001; Manufacturer (none) -> Keystone
- TP201, TP202, TP203: DPN (none) -> 36-5015CT-ND; Distributor (none) -> Digikey; MPN (none) -> 5015; Manufacturer (none) -> Keystone
- U4: DPN (none) -> 296-TPS62912RPURCT-ND; Distributor (none) -> Digikey; MPN (none) -> TPS62912RPUR; Manufacturer (none) -> Texas Instruments
- U7: Distributor (none) -> Digikey; Manufacturer (none) -> Texas Instruments

Commit message: Update documentation for Week 2 Assignment
Parts:
- C218: DPN (none) -> 4713-GMC10X5R335K25NTCT-ND; MPN (none) -> GMC10X5R335K25NT; Manufacturer (none) -> Cal-Chip Electronics, Inc.
- R101, R102, R103, R104, R105: DPN (none) -> P10.0KLCT-ND; MPN (none) -> ERJ-2RKF1002X; Manufacturer (none) -> Panasonic Industry
Changed lines of the file:
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@@
 			)
 		)
-		(property "DPN" ""
+		(property "DPN" "P10.0KLCT-ND"
 			(at 259.08 137.16 90)
 			(effects
@@
 			)
 		)
-		(property "MPN" ""
+		(property "MPN" "ERJ-2RKF1002X"
 			(at 259.08 137.16 90)
 			(effects
@@
 			)
 		)
-		(property "Manufacturer" ""
+		(property "Manufacturer" "Panasonic Industry"
 			(at 259.08 137.16 90)
 			(effects
@@
 			)
 		)
-		(property "DPN" ""
+		(property "DPN" "4713-GMC10X5R335K25NTCT-ND"
 			(at 297.18 110.49 0)
 			(effects
@@
 			)
 		)
-		(property "MPN" ""
+		(property "MPN" "GMC10X5R335K25NT"
 			(at 297.18 110.49 0)
 			(effects
@@
 			)
 		)
-		(property "Manufacturer" ""
+		(property "Manufacturer" "Cal-Chip Electronics, Inc."
 			(at 297.18 110.49 0)
 			(effects
@@
 			)
 		)
-		(property "DPN" ""
+		(property "DPN" "P10.0KLCT-ND"
 			(at 270.51 127 90)
 			(effects
@@
 			)
 		)
-		(property "MPN" ""
+		(property "MPN" "ERJ-2RKF1002X"
 			(at 270.51 127 90)
 			(effects
@@
 			)
 		)
-		(property "Manufacturer" ""
+		(property "Manufacturer" "Panasonic Industry"
 			(at 270.51 127 90)
 			(effects
@@
 			)
 		)
-		(property "DPN" ""
+		(property "DPN" "P10.0KLCT-ND"
 			(at 270.51 137.16 90)
 			(effects
@@
 			)
 		)
-		(property "MPN" ""
+		(property "MPN" "ERJ-2RKF1002X"
 			(at 270.51 137.16 90)
 			(effects
@@
 			)
 		)
-		(property "Manufacturer" ""
+		(property "Manufacturer" "Panasonic Industry"
 			(at 270.51 137.16 90)
 			(effects
@@
 			)
 		)
-		(property "DPN" ""
+		(property "DPN" "P10.0KLCT-ND"
 			(at 241.3 137.16 90)
 			(effects
@@
 			)
 		)
-		(property "MPN" ""
+		(property "MPN" "ERJ-2RKF1002X"
 			(at 241.3 137.16 90)
 			(effects
@@
 			)
 		)
-		(property "Manufacturer" ""
+		(property "Manufacturer" "Panasonic Industry"
 			(at 241.3 137.16 90)
 			(effects
@@
 			)
 		)
-		(property "DPN" ""
+		(property "DPN" "P10.0KLCT-ND"
 			(at 250.19 137.16 90)
 			(effects
@@
 			)
 		)
-		(property "MPN" ""
+		(property "MPN" "ERJ-2RKF1002X"
 			(at 250.19 137.16 90)
 			(effects
@@
 			)
 		)
-		(property "Manufacturer" ""
+		(property "Manufacturer" "Panasonic Industry"
 			(at 250.19 137.16 90)
 			(effects
