File: hardware/Isolated Multi-Rail Power Supply Monitor Sensor Board/Isolated Multi-Rail Power Supply Monitor Sensor Board.kicad_sch (KiCad schematic)
At the start: 70 parts, among them J101 +6VA, J102 +6VB, J103 0039289088, J104 +/-15V, J105 +/-5V, J106 39289108, J107 39289108, J108 Conn_01x04, U4 TPS62912, U5 TCA9803, U6 TCA9803, U7 P82715DR

Commit message: Nightly commit
Parts:
- C18: now in the parts list
- R21: DPN P4.70KLDKR-ND -> 541-0.0JDKR-ND; MPN ERJ-2RKF4701X -> CRCW04020000Z0ED; Manufacturer Panasonic Industry -> Vishay Dale
- R22: footprint Resistor_SMD:R_0402_1005Metric_Pad0.72x0.64mm_HandSolder -> Resistor_SMD:R_0402_1005Metric; now in the parts list
- R23, R24: DPN P4.70KLDKR-ND -> 541-4.70KLCT-ND; MPN ERJ-2RKF4701X -> CRCW04024K70FKED
- R25: value 15k2 -> 14k7; DPN P4.70KLDKR-ND -> P17731CT-ND; MPN ERJ-2RKF4701X -> ERA-2APB1472X
- R26: value 4k87 -> 4k7; DPN P4.70KLDKR-ND -> P4.7KCPCT-ND; MPN ERJ-2RKF4701X -> ERA-2ARB472X
- R27, R28, R29, R30, R31, R32: DPN P4.70KLDKR-ND -> 541-4.70KLCT-ND; MPN ERJ-2RKF4701X -> CRCW04024K70FKED; Manufacturer Panasonic Industry -> Vishay Dale
- TP1, TP3: value TestPoint_Alt -> 5000; DPN (none) -> 36-5000-ND; Distributor (none) -> Digikey; MPN (none) -> 5000; Manufacturer (none) -> Keystone
- TP2: value TestPoint_Alt -> 5001; DPN (none) -> 36-5001-ND; Distributor (none) -> Digikey; MPN (none) -> 5001; Manufacturer (none) -> Keystone
- TP4, TP5, TP6, TP7, TP8, TP9: value TestPoint_Alt -> 5015; DPN (none) -> 36-5015CT-ND; Distributor (none) -> Digikey; MPN (none) -> 5015; Manufacturer (none) -> Keystone
- U4: DPN (none) -> 595-TPS62912RPUR; Distributor (none) -> Mouser; MPN (none) -> TPS62912RPUR; Manufacturer (none) -> Texas Instruments
- U7: DISTRIBUTOR Digikey -> (none); Distributor (none) -> Digikey; Manufacturer (none) -> Texas Instruments

Commit message: Updating for Week 3 Assignment
Parts:
- J101: value +6VA -> +5VA
- J102: value +6VB -> +5VB
Connections:
- net +6VA renamed +5VA
- net +6VA_OUT renamed +5VA_OUT
- net +6VB renamed +5VB
- net +6VB_OUT renamed +5VB_OUT
- net 6VA_SCL renamed 5VA_SCL
- net 6VA_SDA renamed 5VA_SDA
Changed lines of the file:
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@@
 		)
 	)
-	(text_box "6VA MONITORS"
+	(text_box "5VA MONITORS"
 		(exclude_from_sim no)
 		(at 87.63 62.23 0)
@@
 		)
 	)
-	(text_box "6VB MONITORS"
+	(text_box "5VB MONITORS"
 		(exclude_from_sim no)
 		(at 195.58 62.23 0)
@@
 		)
 	)
-	(label "6VB_SDA"
+	(label "5VB_SDA"
 		(at 273.05 82.55 180)
 		(effects
@@
 		)
 	)
-	(label "6VA_SCL"
+	(label "5VA_SCL"
 		(at 383.54 81.28 180)
 		(effects
@@
 		)
 	)
-	(label "+6VB_OUT"
+	(label "+5VB_OUT"
 		(at 33.02 166.37 0)
 		(effects
@@
 		)
 	)
-	(label "6VB_SCL"
+	(label "5VB_SCL"
 		(at 383.54 83.82 180)
 		(effects
@@
 		)
 	)
-	(label "6VA_SDA"
+	(label "5VA_SDA"
 		(at 168.91 82.55 180)
 		(effects
@@
 		)
 	)
-	(label "+6VB_OUT"
+	(label "+5VB_OUT"
 		(at 152.4 15.24 270)
 		(effects
@@
 		)
 	)
-	(label "+6VA_OUT"
+	(label "+5VA_OUT"
 		(at 156.21 68.58 180)
 		(effects
@@
 		)
 	)
-	(label "+6VA_OUT"
+	(label "+5VA_OUT"
 		(at 74.93 166.37 180)
 		(effects
@@
 		)
 	)
-	(label "6VA_SCL"
+	(label "5VA_SCL"
 		(at 168.91 85.09 180)
 		(effects
@@
 		)
 	)
-	(label "+6VA_OUT"
+	(label "+5VA_OUT"
 		(at 143.51 15.24 270)
 		(effects
@@
 		)
 	)
-	(label "6VB_SDA"
+	(label "5VB_SDA"
 		(at 383.54 88.9 180)
 		(effects
@@
 		)
 	)
-	(label "+6VB_OUT"
+	(label "+5VB_OUT"
 		(at 260.35 68.58 180)
 		(effects
@@
 		)
 	)
-	(label "+6VA_OUT"
+	(label "+5VA_OUT"
 		(at 69.85 204.47 180)
 		(effects
@@
 		)
 	)
-	(label "6VB_SCL"
+	(label "5VB_SCL"
 		(at 273.05 85.09 180)
 		(effects
@@
 		)
 	)
-	(label "6VA_SDA"
+	(label "5VA_SDA"
 		(at 383.54 86.36 180)
 		(effects
@@
 		)
 	)
-	(label "+6VB_OUT"
+	(label "+5VB_OUT"
 		(at 27.94 204.47 0)
 		(effects
@@
 	)
 	(symbol
+		(lib_name "+12VA_1")
 		(lib_id "power:+12VA")
 		(at 120.65 67.31 0)
@@
 			)
 		)
-		(property "Value" "+6VA"
+		(property "Value" "+5VA"
 			(at 120.65 63.5 0)
 			(effects
@@
 			)
 		)
-		(property "Value" "+6VA"
+		(property "Value" "+5VA"
 			(at 39.37 93.98 0)
 			(effects
@@
 			)
 		)
-		(property "Value" "+6VB"
+		(property "Value" "+5VB"
 			(at 40.64 119.38 0)
 			(effects
@@
 	)
 	(symbol
+		(lib_name "+12VB_1")
 		(lib_id "+12vb:+12VB")
 		(at 224.79 67.31 0)
@@
 			)
 		)
-		(property "Value" "+6VB"
+		(property "Value" "+5VB"
 			(at 224.79 63.5 0)
 			(effects
@@
 			)
 		)
-		(property "Value" "+6VB"
+		(property "Value" "+5VB"
 			(at 33.02 123.19 0)
 			(effects
@@
 			)
 		)
-		(property "Value" "+6VA"
+		(property "Value" "+5VA"
 			(at 31.75 97.79 0)
 			(effects
